File: kicad/Quorum-Reborn/Quorum-Reborn.kicad_pcb (KiCad board)
At the start: 2 copper layers, 256 parts, among them X1 IN, X10 KEYBOARD 2, X11 SPEAKER, X2 OUT, X3 RGB+TV, X4 SINCLAIR, X6 KEMPSTON, X8 CENTRONICS, X9 KEYBOARD 1

Commit message: Добавлен вариант прошивки Magic-05, в reborn добавлены блокирующие C
Parts:
- removed *DD48: КР1533ЛЕ4, Package_DIP:DIP-14_W7.62mm_Socket_LongPads
- added C102: 0.1, Capacitor_THT:C_Rect_L7.0mm_W2.5mm_P5.00mm, F.Cu at (225.8, 166.5)
- added C103: 0.1, Capacitor_THT:C_Rect_L7.0mm_W2.5mm_P5.00mm, F.Cu at (236.3, 160.2)
- added C104: 0.1, Capacitor_THT:C_Rect_L7.0mm_W2.5mm_P5.00mm, F.Cu at (249.3, 142.5)
- added C107: 0.1, Capacitor_THT:C_Rect_L7.0mm_W2.5mm_P5.00mm, F.Cu at (244.9, 159.8)
- added C108: 0.1, Capacitor_THT:C_Rect_L7.0mm_W2.5mm_P5.00mm, F.Cu at (250.2, -145.4)
- added C130: 0.1, Capacitor_THT:C_Rect_L7.0mm_W2.5mm_P5.00mm, F.Cu at (257.8, 146.6)
- added C131: 0.1, Capacitor_THT:C_Rect_L7.0mm_W2.5mm_P5.00mm, F.Cu at (268.4, 133.1)
- added C132: 0.1, Capacitor_THT:C_Rect_L7.0mm_W2.5mm_P5.00mm, F.Cu at (256.6, 150.6)
- added C133: 0.1, Capacitor_THT:C_Rect_L7.0mm_W2.5mm_P5.00mm, F.Cu at (268.4, 137.1)
- added C134: 0.1, Capacitor_THT:C_Rect_L7.0mm_W2.5mm_P5.00mm, F.Cu at (244.9, 163.8)
- added C135: 0.1, Capacitor_THT:C_Rect_L7.0mm_W2.5mm_P5.00mm, F.Cu at (266.4, 141.2)
- added C136: 0.1, Capacitor_THT:C_Rect_L7.0mm_W2.5mm_P5.00mm, F.Cu at (253.4, 156.6)
- added C137: 0.1, Capacitor_THT:C_Rect_L7.0mm_W2.5mm_P5.00mm, F.Cu at (266.4, 145.2)
- added C202: 0.1, Capacitor_THT:C_Rect_L7.0mm_W2.5mm_P5.00mm, F.Cu at (244.9, 167.9)
- added C206: 0.1, Capacitor_THT:C_Rect_L7.0mm_W2.5mm_P5.00mm, F.Cu at (276.9, 133.1)
- added C207: 0.1, Capacitor_THT:C_Rect_L7.0mm_W2.5mm_P5.00mm, F.Cu at (265.2, 150.6)
- added C208: 0.1, Capacitor_THT:C_Rect_L7.0mm_W2.5mm_P5.00mm, F.Cu at (276.9, 137.1)
- added C209: 0.1, Capacitor_THT:C_Rect_L7.0mm_W2.5mm_P5.00mm, F.Cu at (236.3, 164.2)
- added C210: 0.1, Capacitor_THT:C_Rect_L7.0mm_W2.5mm_P5.00mm, F.Cu at (282.3, 149.3)
- added C211: 0.1, Capacitor_THT:C_Rect_L7.0mm_W2.5mm_P5.00mm, F.Cu at (262.0, 154.7)
- added C212: 0.1, Capacitor_THT:C_Rect_L7.0mm_W2.5mm_P5.00mm, F.Cu at (253.4, 164.7)
- added C214: 0.1, Capacitor_THT:C_Rect_L7.0mm_W2.5mm_P5.00mm, F.Cu at (285.5, 133.1)
- added C217: 0.1, Capacitor_THT:C_Rect_L7.0mm_W2.5mm_P5.00mm, F.Cu at (274.9, 145.2)
- added C218: 0.1, Capacitor_THT:C_Rect_L7.0mm_W2.5mm_P5.00mm, F.Cu at (262.0, 158.7)
- added C220: 0.1, Capacitor_THT:C_Rect_L7.0mm_W2.5mm_P5.00mm, F.Cu at (273.7, 149.3)
- added C221: 0.1, Capacitor_THT:C_Rect_L7.0mm_W2.5mm_P5.00mm, F.Cu at (285.5, 137.1)
- added C222: 0.1, Capacitor_THT:C_Rect_L7.0mm_W2.5mm_P5.00mm, F.Cu at (253.4, 168.8)
- added C226: 0.1, Capacitor_THT:C_Rect_L7.0mm_W2.5mm_P5.00mm, F.Cu at (283.5, 141.2)
- added C227: 0.1, Capacitor_THT:C_Rect_L7.0mm_W2.5mm_P5.00mm, F.Cu at (270.5, 154.7)
- added C228: 0.1, Capacitor_THT:C_Rect_L7.0mm_W2.5mm_P5.00mm, F.Cu at (262.0, 162.8)
- added C229: 0.1, Capacitor_THT:C_Rect_L7.0mm_W2.5mm_P5.00mm, F.Cu at (274.9, 141.2)
- added C239: 0.1, Capacitor_THT:C_Rect_L7.0mm_W2.5mm_P5.00mm, F.Cu at (270.5, 158.7)
- added C242: 0.1, Capacitor_THT:C_Rect_L7.0mm_W2.5mm_P5.00mm, F.Cu at (262.0, 166.8)
- added C245: 0.1, Capacitor_THT:C_Rect_L7.0mm_W2.5mm_P5.00mm, F.Cu at (253.4, 160.7)
- added C246: 0.1, Capacitor_THT:C_Rect_L7.0mm_W2.5mm_P5.00mm, F.Cu at (279.1, 153.3)
- added C247: 0.1, Capacitor_THT:C_Rect_L7.0mm_W2.5mm_P5.00mm, F.Cu at (270.5, 162.8)
- added C249: 0.1, Capacitor_THT:C_Rect_L7.0mm_W2.5mm_P5.00mm, F.Cu at (279.1, 157.4)
- added C250: 0.1, Capacitor_THT:C_Rect_L7.0mm_W2.5mm_P5.00mm, F.Cu at (270.5, 166.8)
- added C251: 0.1, Capacitor_THT:C_Rect_L7.0mm_W2.5mm_P5.00mm, F.Cu at (287.6, 153.3)
- added C30: 0.1, Capacitor_THT:C_Rect_L7.0mm_W2.5mm_P5.00mm, F.Cu at (279.1, 165.5)
- added C31: 0.1, Capacitor_THT:C_Rect_L7.0mm_W2.5mm_P5.00mm, F.Cu at (283.5, 145.2)
- added C32: 0.1, Capacitor_THT:C_Rect_L7.0mm_W2.5mm_P5.00mm, F.Cu at (257.8, 142.5)
- added C33: 0.1, Capacitor_THT:C_Rect_L7.0mm_W2.5mm_P5.00mm, F.Cu at (259.8, 137.1)
- added C34: 0.1, Capacitor_THT:C_Rect_L7.0mm_W2.5mm_P5.00mm, F.Cu at (248.1, 152.6)
- added C35: 0.1, Capacitor_THT:C_Rect_L7.0mm_W2.5mm_P5.00mm, F.Cu at (237.5, 155.7)
- added C36: 0.1, Capacitor_THT:C_Rect_L7.0mm_W2.5mm_P5.00mm, F.Cu at (249.3, 146.6)
- added C37: 0.1, Capacitor_THT:C_Rect_L7.0mm_W2.5mm_P5.00mm, F.Cu at (259.8, 133.1)
- added C4: 0.47, Capacitor_THT:C_Rect_L7.0mm_W2.5mm_P5.00mm, F.Cu at (234.3, 168.3)
- added C5: 0.47, Capacitor_THT:C_Rect_L7.0mm_W2.5mm_P5.00mm, F.Cu at (287.6, 157.4)
- added DD40: КР1533ИР22, Package_DIP:DIP-20_W7.62mm_Socket_LongPads, F.Cu at (226.1, 133.2)
- added DD54: КР1533ЛН1, Package_DIP:DIP-14_W7.62mm_Socket_LongPads, F.Cu at (237.8, 133.2)
- added R19: 1k, Resistor_THT:R_Axial_DIN0204_L3.6mm_D1.6mm_P7.62mm_Horizontal, F.Cu at (249.0, 138.9)
- added R20: 1k, Resistor_THT:R_Axial_DIN0204_L3.6mm_D1.6mm_P7.62mm_Horizontal, F.Cu at (225.5, 162.9)
- added R27: 2k2, Resistor_THT:R_Axial_DIN0204_L3.6mm_D1.6mm_P7.62mm_Horizontal, F.Cu at (249.0, 135.8)
- added R28: 2k2, Resistor_THT:R_Axial_DIN0204_L3.6mm_D1.6mm_P7.62mm_Horizontal, F.Cu at (237.2, 152.1)
- added R34: 2k2, Resistor_THT:R_Axial_DIN0204_L3.6mm_D1.6mm_P7.62mm_Horizontal, F.Cu at (249.0, 132.6)
- added R35: 2k2, Resistor_THT:R_Axial_DIN0204_L3.6mm_D1.6mm_P7.62mm_Horizontal, F.Cu at (225.5, 159.7)
- added X7: COPY OUT, reborn:Jack_3.5mm_Switronic_ST-005-G_horizontal, F.Cu at (14.6, 57.8)
- X1: value IN -> MAG IN; footprint Connectors:DIN5-RA-PTH -> reborn:Jack_3.5mm_Switronic_ST-005-G_horizontal
- X2: value OUT -> MAG OUT; footprint Connectors:DIN5-RA-PTH -> reborn:Jack_3.5mm_Switronic_ST-005-G_horizontal
- moved DD8 317.8 mm to (250.2, -132.7), turned to 90 degrees
- moved X4 315.9 mm to (232.9, -151.8), turned to 180 degrees
- moved X6 291.3 mm to (267.2, -151.8), turned to 180 degrees
- moved ZQ1 254.9 mm to (-19.0, 63.1)
- moved DD41 199.2 mm to (132.1, -139.7)
- moved DD25 167.0 mm to (97.8, -142.2)
- moved X3 150.3 mm to (-7.62, 112.4)
- moved X1 117.4 mm to (14.6, 44.5)
- moved X9 107.5 mm to (-26.0, 122.6)
- moved X2 96.3 mm to (15.2, 69.2)
- moved X10 76.3 mm to (-34.9, 122.6)
Connections:
- DD104 pad 11: Net-(DD104-Pad10) -> /~RDFF
- DD104 pad 12: Net-(DD104-Pad10) -> /BORD
- DD108 pad 3: (no net) -> Net-(DD108-Pad3)
- DD108 pad 38: (no net) -> Net-(DD108-Pad38)
- DD108 pad 4: (no net) -> Net-(DD108-Pad4)
- DD23 pad 5: Net-(DD104-Pad13) -> Net-(DD23-Pad5)
- DD3 pad 12: (no net) -> /~RDFF
- DD43 pad 12: Net-(*DD48-Pad1) -> Net-(DD43-Pad12)
- DD48 pad 1: (no net) -> Net-(DD43-Pad12)
- DD48 pad 10: (no net) -> /R
- DD48 pad 11: (no net) -> /B
- DD48 pad 12: (no net) -> Net-(DD48-Pad12)
- DD48 pad 13: (no net) -> GND
- DD48 pad 2: (no net) -> GND
- DD48 pad 3: (no net) -> Net-(DD48-Pad12)
- DD48 pad 4: (no net) -> Net-(DD48-Pad12)
- DD48 pad 5: (no net) -> Net-(DD48-Pad5)
- DD48 pad 6: (no net) -> /Y
- DD48 pad 8: (no net) -> Net-(DD48-Pad5)
- DD48 pad 9: (no net) -> /G
- R70 pad 2: Net-(*DD48-Pad1) -> Net-(DD43-Pad12)
- X2 pad 1: /MIC -> (no net)
Routing:
- net /D5: track 0.00 -> 66.9 mm
- net /D4: track 0.00 -> 56.9 mm
- net /D3: track 0.00 -> 56.9 mm
- net /A13: track 0.00 -> 53.6 mm, vias 0 -> 1
- net /A10: track 0.00 -> 53.5 mm, vias 0 -> 2
- net /D6: track 0.00 -> 52.6 mm, vias 0 -> 1
- net /D7: track 0.00 -> 51.6 mm
- net /A9: track 0.00 -> 41.0 mm, vias 0 -> 1
- net /D2: track 0.00 -> 36.4 mm, vias 0 -> 1
- net /D1: track 0.00 -> 36.4 mm
- net /D0: track 0.00 -> 36.4 mm
- net /A8: track 0.00 -> 36.4 mm
- net /A12: track 0.00 -> 35.3 mm
- net /KEMPL: track 0.00 -> 20.6 mm
- net /KEMPR: track 0.00 -> 20.5 mm
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Other:
- net class Power added: clearance 0.2, trace_width 0.7, via_dia 0.8, via_drill 0.4
