File: kicad/Quorum-BK04/Quorum-BK04-mods.sch (KiCad schematic (older format))
At the start: 232 parts, among them X1 SINCLAIR, X10 RGB, X11 TAPE OUT, X12 CENTRONICS, X2 KEMPSTON, X3 KEYBOARD 1, X4 KEYBOARD 2, X5 TAPE IN, X6.1 EXPANSION B, X6.2 EXPANSION A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

Commit message: BK04: Исправлены ошибки, добавлен вариант с модификациями
Parts:
- added *DD101: КР1533ИР22, Package_DIP:DIP-20_W7.62mm_Socket_LongPads, symbol ics_gost:ИР22
- added *DD102: КР1533ЛЛ1, Package_DIP:DIP-14_W7.62mm_Socket_LongPads, symbol ics_gost:ЛЛ1
- added *DD103: КР1533ЛИ1, Package_DIP:DIP-14_W7.62mm_Socket_LongPads, symbol ics_gost:ЛИ1
- added *DD104: КР1533ЛЕ1, Package_DIP:DIP-14_W7.62mm_Socket_LongPads, symbol ics_gost:ЛЕ1
- added unit 4 of DD52
- added KT7, KT8, KT9: TestPoint, TestPoint:TestPoint_THTPad_D1.5mm_Drill0.7mm, symbol Connector:TestPoint
- added S1: TURBO, symbol gost_common:SWITCH
- renumbered DA4 to DD4, DA51 to DD51
Connections:
- net labels added: CLK, ~RDFF
- wire segments 1589 -> 1635
- no-connect marks 39 -> 38
Other:
- note added: "*Pentagon"
