File: kicad/Quorum-BK04/Quorum-BK04-mods.sch (KiCad schematic (older format))
At the start: 240 parts, among them X1 SINCLAIR, X10 RGB, X11 TAPE OUT, X12 CENTRONICS, X2 KEMPSTON, X3 KEYBOARD 1, X4 KEYBOARD 2, X5 TAPE IN, X6.1 EXPANSION B, X6.2 EXPANSION A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

Commit message: Мелкие правки
Parts:
- VT1, VT2, VT3, VT4, VT6, VT7: symbol ics_gost:VT_NPN_EBC -> gost_common:VT_NPN_EBC
- VT5: symbol ics_gost:VT_PNP_EBC -> gost_common:VT_PNP_EBC
Changed lines of the file:
@@
 UncleRus
 $Comp
-L ics_gost:VT_NPN_EBC VT6
+L gost_common:VT_NPN_EBC VT6
 U 1 1 5E90BEA2
 P 26200 15700
@@
 $EndComp
 $Comp
-L ics_gost:VT_PNP_EBC VT5
+L gost_common:VT_PNP_EBC VT5
 U 1 1 BC44D7BF
 P 26200 16100
@@
 	22550 12350 22400 12350
 $Comp
-L ics_gost:VT_NPN_EBC VT1
+L gost_common:VT_NPN_EBC VT1
 U 1 1 9473CEF6
 P 23550 12350
@@
 $EndComp
 $Comp
-L ics_gost:VT_NPN_EBC VT3
+L gost_common:VT_NPN_EBC VT3
 U 1 1 95557F79
 P 23550 13650
@@
 $EndComp
 $Comp
-L ics_gost:VT_NPN_EBC VT2
+L gost_common:VT_NPN_EBC VT2
 U 1 1 95952913
 P 23550 13000
@@
 	20300 3400 20300 5100
 $Comp
-L ics_gost:VT_NPN_EBC VT7
+L gost_common:VT_NPN_EBC VT7
 U 1 1 A56AA70A
 P 21150 15800
@@
 $EndComp
 $Comp
-L ics_gost:VT_NPN_EBC VT4
+L gost_common:VT_NPN_EBC VT4
 U 1 1 C6A0C03A
 P 25200 17350

Commit message: BK04: мелкие правки
Parts:
- VD1, VD2, VD3, VD4, VD5, VD6, VD7, VD8: symbol Device:D -> gost_common:DIODE
Changed lines of the file:
@@
 $EndComp
 $Comp
-L Device:D VD1
+L gost_common:DIODE VD1
 U 1 1 5E90BCE0
 P 6700 16400
@@
 	5800 16400 6550 16400
 $Comp
-L Device:D VD2
+L gost_common:DIODE VD2
 U 1 1 5DDFFBE8
 P 6850 16300
@@
 $EndComp
 $Comp
-L Device:D VD3
+L gost_common:DIODE VD3
 U 1 1 5E90BCEA
 P 6700 16200
@@
 $EndComp
 $Comp
-L Device:D VD4
+L gost_common:DIODE VD4
 U 1 1 5E90BCEB
 P 6850 16100
@@
 $EndComp
 $Comp
-L Device:D VD5
+L gost_common:DIODE VD5
 U 1 1 5E90BCEE
 P 6700 16000
@@
 	5800 16000 6550 16000
 $Comp
-L Device:D VD6
+L gost_common:DIODE VD6
 U 1 1 5E90BCEF
 P 6850 15900
@@
 $EndComp
 $Comp
-L Device:D VD7
+L gost_common:DIODE VD7
 U 1 1 5DE1BA8A
 P 6700 15800
@@
 	5800 15800 6550 15800
 $Comp
-L Device:D VD8
+L gost_common:DIODE VD8
 U 1 1 5DE1BA95
 P 6850 15700

Commit message: Q64: добавлен вариант модификаций, DD: плата
Connections:
- net labels removed: SOUND
- wire segments 1635 -> 1633
Changed lines of the file:
@@
 Entry Bus Bus
 	20650 11800 20550 11900
-Entry Wire Line
-	24800 15300 24900 15200
-Text Label 24900 15100 0    50   ~ 0
-MIC
 $Comp
 L gost_common:CONN_6_R X11
@@
 	1    0    0    -1
 $EndComp
-$Comp
-L gost_common:RESISTOR R47
-U 1 1 B6F43CBE
-P 25950 15450
-F 0 "R47" V 25904 15521 50  0000 L CNN
-F 1 "10k" V 25995 15521 50  0000 L CNN
-F 2 "Resistor_THT:R_Axial_DIN0204_L3.6mm_D1.6mm_P7.62mm_Horizontal" H 25950 15450 0   0001 C CNN
-F 3 "" H 25950 15450 50  0001 C CNN
-	1    25950 15450
-	0    1    1    0
-$EndComp
-Entry Wire Line
-	24800 15200 24900 15100
-Text Label 24900 15200 0    50   ~ 0
-SPK
-Wire Wire Line
-	25950 15300 25950 15100
-Wire Wire Line
-	25650 15200 25650 15300
-Wire Wire Line
-	25650 15600 25650 15700
-Wire Wire Line
-	25950 15700 25950 15600
-Wire Wire Line
-	25650 15700 25950 15700
-Wire Wire Line
-	25550 15700 25650 15700
-Connection ~ 25650 15700
-Wire Wire Line
-	24900 15100 25950 15100
-Wire Wire Line
-	24900 15200 25650 15200
 Text Label 24900 15700 0    50   ~ 0
 COPY
@@
 Wire Wire Line
 	24900 15700 25250 15700
-Wire Wire Line
-	25950 15700 26100 15700
-Connection ~ 25950 15700
 Text Label 24900 16100 0    50   ~ 0
 USP
@@
 	-1   0    0    1
 $EndComp
-$Comp
-L gost_common:RESISTOR R46
-U 1 1 B6F44D1D
-P 25650 15450
-F 0 "R46" V 25604 15521 50  0000 L CNN
-F 1 "1k" V 25695 15521 50  0000 L CNN
-F 2 "Resistor_THT:R_Axial_DIN0204_L3.6mm_D1.6mm_P7.62mm_Horizontal" H 25650 15450 0   0001 C CNN
-F 3 "" H 25650 15450 50  0001 C CNN
-	1    25650 15450
-	0    1    1    0
-$EndComp
 Wire Wire Line
 	27850 15350 27750 15350
@@
 Wire Wire Line
 	27350 15850 27200 15850
-Wire Wire Line
-	27200 16650 24900 16650
 Connection ~ 27350 15850
 Wire Wire Line
 	27350 15850 27350 15750
-Entry Wire Line
-	24800 16750 24900 16650
-Text Label 24900 16650 0    50   ~ 0
-SOUND
-Wire Wire Line
-	27200 15850 27200 16650
-Text Label 24900 16750 0    50   ~ 0
-MIC
-Entry Wire Line
-	24800 16850 24900 16750
-Wire Wire Line
-	24900 16750 25550 16750
 $Comp
 L gost_common:RESISTOR R48
@@
 Wire Wire Line
 	27850 18050 27200 18050
-Wire Wire Line
-	27200 18050 27200 16650
-Connection ~ 27200 16650
 $Comp
 L gost_common:+5V #PWR0162
@@
 	21850 18100 21750 18100
 Connection ~ 21750 18100
-$Comp
-L ics_gost:ИР22 *DD101
-U 1 1 5F3C5DC3
-P 19250 9000
-F 0 "*DD101" H 19250 9768 50  0000 C CNN
-F 1 "КР1533ИР22" H 19250 9677 50  0000 C CNN
-F 2 "Package_DIP:DIP-20_W7.62mm_Socket_LongPads" H 19350 9600 50  0001 C CNN
-F 3 "" H 19350 9600 50  0001 C CNN
-F 4 "*port FF" H 19250 8050 50  0000 C CIN "Note"
-	1    19250 9000
-	1    0    0    -1
-$EndComp
-$Comp
-L gost_common:+5V #PWR0168
-U 1 1 5F3ED26A
-P 18450 9700
-F 0 "#PWR0168" H 18450 9670 50  0001 C TNN
-F 1 "+5V" V 18450 9831 50  0000 L CNN
-F 2 "" H 18450 9700 0   0001 C CNN
-F 3 "" H 18450 9700 50  0001 C CNN
-	1    18450 9700
-	0    -1   -1   0
-$EndComp
-$Comp
-L gost_common:GND #PWR0169
-U 1 1 5F3ED274
-P 18750 9800
-F 0 "#PWR0169" H 18750 9830 50  0001 C BNN
-F 1 "GND" H 18750 9670 50  0001 C TNN
-F 2 "" H 18750 9800 0   0001 C CNN
-F 3 "" H 18750 9800 50  0001 C CNN
-	1    18750 9800
-	1    0    0    -1
-$EndComp
-Entry Wire Line
-	17800 10350 17900 10250
-Text Label 17900 10250 0    50   ~ 0
-BORD
-Entry Wire Line
-	17800 10250 17900 10150
-Text Label 17900 10150 0    50   ~ 0
-~RDFF
-Wire Wire Line
-	18600 10000 18600 9500
-Wire Wire Line
-	18600 9500 18750 9500
 Entry Wire Line
 	18300 8500 18200 8400
@@
 Text Label 18300 9200 0    50   ~ 0
 MD7
-Wire Wire Line
-	18300 8500 18750 8500
-Wire Wire Line
-	18300 8600 18750 8600
-Wire Wire Line
-	18300 8700 18750 8700
-Wire Wire Line
-	18300 8800 18750 8800
-Wire Wire Line
-	18300 8900 18750 8900
-Wire Wire Line
-	18300 9000 18750 9000
-Wire Wire Line
-	18300 9100 18750 9100
-Wire Wire Line
-	18300 9200 18750 9200
 Entry Wire Line
 	20550 8600 20450 8500
@@
 Text Label 20450 9200 2    50   ~ 0
 D7
-Wire Wire Line
-	19750 8500 20450 8500
-Wire Wire Line
-	19750 8600 20450 8600
-Wire Wire Line
-	19750 8700 20450 8700
-Wire Wire Line
-	19750 8800 20450 8800
-Wire Wire Line
-	19750 8900 20450 8900
-Wire Wire Line
-	19750 9000 20450 9000
-Wire Wire Line
-	19750 9100 20450 9100
-Wire Wire Line
-	19750 9200 20450 9200
-Wire Wire Line
-	18450 9700 18750 9700
 Entry Wire Line
 	17800 9500 17900 9400
 Text Label 17900 9400 0    50   ~ 0
 DC2
-Wire Wire Line
-	17900 9400 18750 9400
-Wire Wire Line
-	18800 10000 18600 10000
-Wire Wire Line
-	17900 10250 18200 10250
-Wire Wire Line
-	17900 10150 18200 10150
-$Comp
-L ics_gost:ЛЛ1 *DD102
-U 1 1 5F3D32A7
-P 18500 10200
-F 0 "*DD102" H 18500 10025 50  0000 C CNN
-F 1 "КР1533ЛЛ1" H 18500 9934 50  0000 C CNN
-F 2 "Package_DIP:DIP-14_W7.62mm_Socket_LongPads" H 18550 10350 50  0001 C CNN
-F 3 "" H 18550 10350 50  0001 C CNN
-	1    18500 10200
-	1    0    0    -1
-$EndComp
-Wire Wire Line
-	18800 10000 18800 10150
 $Comp
 L ics_gost:ЛЛ1 *DD102
@@
 	0    1    -1   0
 $EndComp
+$Comp
+L gost_common:+5V #PWR0168
+U 1 1 5F3ED26A
+P 18450 9700
+F 0 "#PWR0168" H 18450 9670 50  0001 C TNN
+F 1 "+5V" V 18450 9831 50  0000 L CNN
+F 2 "" H 18450 9700 0   0001 C CNN
+F 3 "" H 18450 9700 50  0001 C CNN
+	1    18450 9700
+	0    -1   -1   0
+$EndComp
+Wire Wire Line
+	17900 10150 18200 10150
+Wire Wire Line
+	17900 10250 18200 10250
+Text Label 17900 10150 0    50   ~ 0
+~RDFF
+Entry Wire Line
+	17800 10250 17900 10150
+Text Label 17900 10250 0    50   ~ 0
+BORD
+Entry Wire Line
+	17800 10350 17900 10250
+Wire Wire Line
+	18800 10000 18800 10150
+Wire Wire Line
+	18800 10000 18600 10000
+Wire Wire Line
+	18600 10000 18600 9500
+$Comp
+L ics_gost:ЛЛ1 *DD102
+U 1 1 5F3D32A7
+P 18500 10200
+F 0 "*DD102" H 18500 10025 50  0000 C CNN
+F 1 "КР1533ЛЛ1" H 18500 9934 50  0000 C CNN
+F 2 "Package_DIP:DIP-14_W7.62mm_Socket_LongPads" H 18550 10350 50  0001 C CNN
+F 3 "" H 18550 10350 50  0001 C CNN
+	1    18500 10200
+	1    0    0    -1
+$EndComp
+Wire Wire Line
+	19750 8800 20450 8800
+Wire Wire Line
+	18300 8800 18750 8800
+Wire Wire Line
+	18300 8700 18750 8700
+Wire Wire Line
+	19750 8700 20450 8700
+Wire Wire Line
+	19750 8600 20450 8600
+Wire Wire Line
+	18300 8600 18750 8600
+Wire Wire Line
+	18300 8500 18750 8500
+Wire Wire Line
+	19750 8500 20450 8500
+Wire Wire Line
+	19750 9200 20450 9200
+Wire Wire Line
+	18300 9200 18750 9200
+Wire Wire Line
+	18300 9100 18750 9100
+Wire Wire Line
+	19750 9100 20450 9100
+Wire Wire Line
+	19750 9000 20450 9000
+Wire Wire Line
+	18300 9000 18750 9000
+Wire Wire Line
+	18300 8900 18750 8900
+Wire Wire Line
+	19750 8900 20450 8900
+Wire Wire Line
+	17900 9400 18750 9400
+Wire Wire Line
+	18600 9500 18750 9500
+Wire Wire Line
+	18450 9700 18750 9700
+$Comp
+L gost_common:GND #PWR0169
+U 1 1 5F3ED274
+P 18750 9800
+F 0 "#PWR0169" H 18750 9830 50  0001 C BNN
+F 1 "GND" H 18750 9670 50  0001 C TNN
+F 2 "" H 18750 9800 0   0001 C CNN
+F 3 "" H 18750 9800 50  0001 C CNN
+	1    18750 9800
+	1    0    0    -1
+$EndComp
+$Comp
+L ics_gost:ИР22 *DD101
+U 1 1 5F3C5DC3
+P 19250 9000
+F 0 "*DD101" H 19250 9768 50  0000 C CNN
+F 1 "КР1533ИР22" H 19250 9677 50  0000 C CNN
+F 2 "Package_DIP:DIP-20_W7.62mm_Socket_LongPads" H 19350 9600 50  0001 C CNN
+F 3 "" H 19350 9600 50  0001 C CNN
+F 4 "*port FF" H 19250 8050 50  0000 C CIN "Note"
+	1    19250 9000
+	1    0    0    -1
+$EndComp
+Wire Wire Line
+	27200 15850 27200 18050
+Connection ~ 25650 15700
+Wire Wire Line
+	25550 15700 25650 15700
+$Comp
+L gost_common:RESISTOR R46
+U 1 1 B6F44D1D
+P 25650 15450
+F 0 "R46" V 25604 15521 50  0000 L CNN
+F 1 "1k" V 25695 15521 50  0000 L CNN
+F 2 "Resistor_THT:R_Axial_DIN0204_L3.6mm_D1.6mm_P7.62mm_Horizontal" H 25650 15450 0   0001 C CNN
+F 3 "" H 25650 15450 50  0001 C CNN
+	1    25650 15450
+	0    1    1    0
+$EndComp
+Wire Wire Line
+	25650 15600 25650 15700
+Wire Wire Line
+	25650 15200 25650 15300
+Wire Wire Line
+	24900 15200 25650 15200
+Text Label 24900 15200 0    50   ~ 0
+SPK
+Entry Wire Line
+	24800 15300 24900 15200
+Connection ~ 25950 15700
+Wire Wire Line
+	25950 15700 26100 15700
+Wire Wire Line
+	25650 15700 25950 15700
+Wire Wire Line
+	25950 15700 25950 15600
+Wire Wire Line
+	25950 15300 25950 15100
+$Comp
+L gost_common:RESISTOR R47
+U 1 1 B6F43CBE
+P 25950 15450
+F 0 "R47" V 25904 15521 50  0000 L CNN
+F 1 "10k" V 25995 15521 50  0000 L CNN
+F 2 "Resistor_THT:R_Axial_DIN0204_L3.6mm_D1.6mm_P7.62mm_Horizontal" H 25950 15450 0   0001 C CNN
+F 3 "" H 25950 15450 50  0001 C CNN
+	1    25950 15450
+	0    1    1    0
+$EndComp
+Entry Wire Line
+	24800 15200 24900 15100
+Text Label 24900 15100 0    50   ~ 0
+MIC
+Entry Wire Line
+	24800 16850 24900 16750
+Text Label 24900 16750 0    50   ~ 0
+MIC
+Wire Wire Line
+	24900 16750 25550 16750
+Wire Wire Line
+	24900 15100 25950 15100
+Wire Bus Line
+	24800 15000 24800 16850
+Wire Bus Line
+	20550 6200 20550 14900
+Wire Bus Line
+	18200 1800 18200 9100
+Wire Bus Line
+	20800 2100 20800 2900
+Wire Bus Line
+	20150 2100 20150 2800
 Wire Bus Line
 	12700 1800 18200 1800
@@
 	12300 19200 17800 19200
 Wire Bus Line
+	12700 1800 12700 15850
+Wire Bus Line
 	8900 10100 12200 10100
 Wire Bus Line
-	20150 2100 20150 2800
+	8900 2300 8900 10100
 Wire Bus Line
-	20800 2100 20800 2900
+	17800 2400 17800 19200
 Wire Bus Line
-	24800 15000 24800 16850
-Wire Bus Line
-	7450 15800 7450 16950
-Wire Bus Line
-	6350 11700 6350 15400
-Wire Bus Line
-	18200 1800 18200 9100
+	14900 3300 14900 19100
 Wire Bus Line
 	14500 1900 14500 15150
@@
 	12300 2100 12300 19200
 Wire Bus Line
-	20550 6200 20550 14900
+	23550 2300 23550 11800
 Wire Bus Line
 	9750 10200 9750 18250
 Wire Bus Line
-	23550 2300 23550 11800
+	6350 11700 6350 15400
 Wire Bus Line
-	8900 2300 8900 10100
-Wire Bus Line
-	12700 1800 12700 15850
-Wire Bus Line
-	14900 3300 14900 19100
-Wire Bus Line
-	17800 2400 17800 19200
+	7450 15800 7450 16950
 $EndSCHEMATC

Commit message: Обновлены УГО разъемов, исправлены множественные ошибки в схемах клавиатур
Parts:
- X12: NET1 ~STROBE -> /STROBE
- X4: NET12 ~RES~ -> ~RES
- X6.1: NET13 ~IORQGE -> /IORQGE; NET19 ~BUSRQ -> /BUSRQ; NET20 ~RES -> /RES; NET25 ~ROMCS -> /ROMCS; NET26 ~BUSAK -> /BUSAK
- X6.2: NET13 ~INT -> /INT; NET14 ~NMI -> /NMI; NET15 ~HALT~ -> /HALT; NET16 ~MREQ~ -> /MREQ; NET17 ~IORQ -> /IORQ; NET18 ~RD~ -> /RD; NET19 ~WR -> /WR; NET21 ~WAIT~ -> /WAIT; NET24 ~M1~ -> /M1; NET25 ~RFSH~ -> /RFSH; NET28 ~UPS -> /UPS; NET4 ~RAMCS -> /RAMCS
