File: kicad/Quorum-BK04/Quorum-BK04.sch (KiCad schematic (older format))
At the start: 232 parts, among them X1 SINCLAIR, X10 RGB, X11 TAPE OUT, X12 CENTRONICS, X2 KEMPSTON, X3 KEYBOARD 1, X4 KEYBOARD 2, X5 TAPE IN, X6.1 EXPANSION B, X6.2 EXPANSION A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

Commit message: Мелкие правки
Parts:
- VT1, VT2, VT3, VT4, VT6, VT7: symbol ics_gost:VT_NPN_EBC -> gost_common:VT_NPN_EBC
- VT5: symbol ics_gost:VT_PNP_EBC -> gost_common:VT_PNP_EBC
Changed lines of the file:
@@
 UncleRus
 $Comp
-L ics_gost:VT_NPN_EBC VT6
+L gost_common:VT_NPN_EBC VT6
 U 1 1 5E90BEA2
 P 26200 15700
@@
 $EndComp
 $Comp
-L ics_gost:VT_PNP_EBC VT5
+L gost_common:VT_PNP_EBC VT5
 U 1 1 BC44D7BF
 P 26200 16100
@@
 	22550 12350 22400 12350
 $Comp
-L ics_gost:VT_NPN_EBC VT1
+L gost_common:VT_NPN_EBC VT1
 U 1 1 9473CEF6
 P 23550 12350
@@
 $EndComp
 $Comp
-L ics_gost:VT_NPN_EBC VT3
+L gost_common:VT_NPN_EBC VT3
 U 1 1 95557F79
 P 23550 13650
@@
 $EndComp
 $Comp
-L ics_gost:VT_NPN_EBC VT2
+L gost_common:VT_NPN_EBC VT2
 U 1 1 95952913
 P 23550 13000
@@
 	20300 3400 20300 5100
 $Comp
-L ics_gost:VT_NPN_EBC VT7
+L gost_common:VT_NPN_EBC VT7
 U 1 1 A56AA70A
 P 21150 15800
@@
 $EndComp
 $Comp
-L ics_gost:VT_NPN_EBC VT4
+L gost_common:VT_NPN_EBC VT4
 U 1 1 C6A0C03A
 P 25200 17350

Commit message: BK04: мелкие правки
Parts:
- VD1, VD2, VD3, VD4, VD5, VD6, VD7, VD8: symbol Device:D -> gost_common:DIODE
Changed lines of the file:
@@
 $EndComp
 $Comp
-L Device:D VD1
+L gost_common:DIODE VD1
 U 1 1 5E90BCE0
 P 6700 16400
@@
 	5800 16400 6550 16400
 $Comp
-L Device:D VD2
+L gost_common:DIODE VD2
 U 1 1 5DDFFBE8
 P 6850 16300
@@
 $EndComp
 $Comp
-L Device:D VD3
+L gost_common:DIODE VD3
 U 1 1 5E90BCEA
 P 6700 16200
@@
 $EndComp
 $Comp
-L Device:D VD4
+L gost_common:DIODE VD4
 U 1 1 5E90BCEB
 P 6850 16100
@@
 $EndComp
 $Comp
-L Device:D VD5
+L gost_common:DIODE VD5
 U 1 1 5E90BCEE
 P 6700 16000
@@
 	5800 16000 6550 16000
 $Comp
-L Device:D VD6
+L gost_common:DIODE VD6
 U 1 1 5E90BCEF
 P 6850 15900
@@
 $EndComp
 $Comp
-L Device:D VD7
+L gost_common:DIODE VD7
 U 1 1 5DE1BA8A
 P 6700 15800
@@
 	5800 15800 6550 15800
 $Comp
-L Device:D VD8
+L gost_common:DIODE VD8
 U 1 1 5DE1BA95
 P 6850 15700

Commit message: Обновлены УГО разъемов, исправлены множественные ошибки в схемах клавиатур
Parts:
- X12: NET1 ~STROBE -> /STROBE
- X6.1: NET13 ~IORQGE -> /IORQGE; NET19 ~BUSRQ -> /BUSRQ; NET20 ~RES -> /RES; NET25 ~ROMCS -> /ROMCS; NET26 ~BUSAK -> /BUSAK
- X6.2: NET13 ~INT -> /INT; NET14 ~NMI -> /NMI; NET15 ~HALT~ -> /HALT~; NET16 ~MREQ~ -> /MREQ; NET17 ~IORQ -> /IORQ; NET18 ~RD~ -> /RD; NET19 ~WR -> /WR; NET21 ~WAIT~ -> /WAIT; NET24 ~M1~ -> /M1; NET25 ~RFSH~ -> /RFSH; NET28 ~UPS -> /UPS; NET4 ~RAMCS -> /RAMCS
