File: kicad/Quorum-BK04/keyboard.sch (KiCad schematic (older format))
At the start: 90 parts, among them X101 KEYBOARD 1, X102 KEYBOARD 2

Commit message: Обновлены УГО разъемов, исправлены множественные ошибки в схемах клавиатур
Parts:
- removed X101: KEYBOARD 1, symbol gost_common:CONN_12
- removed X102: KEYBOARD 2, symbol gost_common:CONN_12
- added X101: TOP FILM, symbol gost_common:CONN_12_R
- added X102: BOTTOM FILM, symbol gost_common:CONN_12_R
- renumbered S46 to S1, S3 to S10, S4 to S11, S5 to S12, S6 to S13, S7 to S14, S8 to S15, S9 to S16, S53 to S17, S54 to S18, S55 to S19, S47 to S2, S56 to S20, S57 to S21, S58 to S22, S10 to S23, S11 to S24, S12 to S25, S13 to S26, S14 to S27, S15 to S28, S16 to S29, S48 to S3, S17 to S30, S18 to S31, S19 to S32, S20 to S33, S21 to S34, S22 to S35, S23 to S36, S24 to S37, S25 to S38, S26 to S39, S49 to S4, S27 to S40, S28 to S41, S29 to S42, S30 to S43, S31 to S44, S32 to S45, S33 to S46, S34 to S47, S35 to S48, S36 to S49, S50 to S5, S37 to S50, S38 to S51, S39 to S52, S40 to S53, S41 to S54, S42 to S55, S43 to S56, S44 to S57, S45 to S58, S51 to S6, S52 to S7, S1 to S8, S88 to S85, S87 to S86, S86 to S87, S85 to S88, S2 to S9
Connections:
- net labels added: K_D0, K_D0*, K_D1, K_D1*, K_D2, K_D2*, K_D3, K_D3*, K_D4, K_D4*, K_D5*
- net labels removed: KINV, KNMI, KSPK, ~RES
- wire segments 449 -> 453
Other:
- note added: "EDIT"
- note removed: "CAPS\nLOCK"
- note removed: "TAB"
